File: brain-of-pleiades.kicad_sch (KiCad schematic)
At the start: 1 part, among them U1 4078_CD4051B_Analog_Switch

Commit message: fleshing out design
Parts:
- added J1: 3040_Connector_SL_8pos_Vert, Shulltronics_Connectors:3040_Molex_SL_8pos_Vert, symbol Shulltronics_Connectors:3040_Connector_SL_8pos_Vert
- added J2, J3, J4, J7: 3030_Connector_SL_3pos_Vert, Shulltronics_Connectors:3030_Molex_SL_3pos_Vert, symbol Shulltronics_Connectors:3030_Connector_SL_3pos_Vert
- added J5: 4039_Header_Male_Vert_16pin_0.1in, Shulltronics_Connectors:4039_Header_16pos_2.54mm, symbol Shulltronics_Connectors:4039_Header_Male_Vert_16pin_0.1in
- added J6: 4040_Header_Male_Vert_12pin_0.1in, Shulltronics_Connectors:4040_Header_12pos_2.54mm, symbol Shulltronics_Connectors:4040_Header_Male_Vert_12pin_0.1in
- added L1: Shulltronics_Logo, Shulltronics_Generics:Shulltronics_Logo, symbol Shulltronics_Sch_Symbols:Shulltronics_Logo
Connections:
- net at U1.1 (X4): now also J1.5
- net at U1.12 (X3): now also J1.4
- net at U1.13 (X0): now also J1.1
- net at U1.14 (X1): now also J1.2
- net at U1.15 (X2): now also J1.3
- net at U1.2 (X6): now also J1.7
- net at U1.4 (X7): now also J1.8
- net at U1.5 (X5): now also J1.6
- new net A0: J5.12
- new net A1: J5.11
- new net A2: J5.10
- new net A3: J5.9
- new net D10: J6.7
- new net D11: J6.6
- new net D12: J6.5
- new net D13: J6.4
- new net D6: J6.9
- new net D9: J6.8
- new net GND: J5.13
- new net MISO: J5.4
- new net MOSI: J5.5
- new net RX: J5.3
- new net SCK: J5.6
- new net SCL: J6.11
- new net SDA: J6.12
- new net TX: J5.2
- new net USB: J6.3
- new net USER: J5.1
- new net VBAT: J6.1
- new net VREF: J5.14
- new net ~{EN}: J6.2
- new net ~{RST}: J5.16
- no-connect marks 0 -> 23
Other:
- note added: "Analog Inputs & Mux"
- note added: "MIDI Output"
- note added: "NeoPixel Outputs"
- moved on the sheet: U1
